File: Hardware/Kte4402.3/EPROM_BANK.sch (EAGLE design)
At the start: 50 parts, among them IC1 DS8286D, IC10 D8205, IC11 DL000, IC12 DL074, IC13 D8205, IC14 DL000, IC15 D8205, IC2 DL541, IC3 DL541, IC4 DL541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

Commit message: Fehlerhafte Signalbezeichnung
!MDIS wird nicht invertiert . Da IC9 ein EXOR ist ( 0 xor 0 = 0 ; 1 xor
0 = 1)
Connections:
- net MDIS renamed !MDIS_INT
Changed lines of the file:
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@@
 <?xml version="1.0" encoding="utf-8"?>
 <!DOCTYPE eagle SYSTEM "eagle.dtd">
-<eagle version="7.4.0">
+<eagle version="7.6.0">
 <drawing>
 <settings>
@@
 </segment>
 </net>
-<net name="MDIS" class="0">
+<net name="!MDIS_INT" class="0">
 <segment>
 <pinref part="IC9" gate="/1" pin="Y"/>
